Commit message: Remove the lidar and the limits on the shoulder pitch in order to have it running we need to copy the limits in the install folder

File: urdf/ergoCub/robots/ergoCubSN000/model.urdf (robot description, URDF)
Before this commit: robot ergoCub, 169 links, 168 joints
Joints:
- joint camera_tilt: limit lower=-0.5235987755982988 upper=0.5235987755982988 effort=50000 velocity=120.0 -> lower=-3.5235987755982988 upper=3.5235987755982988 effort=50000 velocity=120.0
- joint l_ankle_pitch: limit lower=-0.7853981633974483 upper=0.7853981633974483 effort=50000 velocity=120.0 -> lower=-3.7853981633974483 upper=3.7853981633974483 effort=50000 velocity=120.0
- joint l_ankle_roll: limit lower=-0.4363323129985824 upper=0.4363323129985824 effort=50000 velocity=120.0 -> lower=-3.4363323129985824 upper=3.4363323129985824 effort=50000 velocity=120.0
- joint l_elbow: limit lower=-0.05235987755982989 upper=1.3089969389957472 effort=50000 velocity=120.0 -> lower=-3.05235987755982989 upper=3.3089969389957472 effort=50000 velocity=120.0
- joint l_hip_pitch: limit lower=-0.7853981633974483 upper=2.007128639793479 effort=50000 velocity=120.0 -> lower=-3.7853981633974483 upper=3.007128639793479 effort=50000 velocity=120.0
- joint l_hip_roll: limit lower=-0.6108652381980153 upper=1.9547687622336491 effort=50000 velocity=120.0 -> lower=-3.6108652381980153 upper=3.9547687622336491 effort=50000 velocity=120.0
- joint l_hip_yaw: limit lower=-1.3962634015954636 upper=1.3962634015954636 effort=50000 velocity=120.0 -> lower=-3.3962634015954636 upper=3.3962634015954636 effort=50000 velocity=120.0
- joint l_index_add: limit lower=0.0 upper=0.3490658503988659 effort=50000 velocity=120.0 -> lower=0.0 upper=3.3490658503988659 effort=50000 velocity=120.0
- joint l_index_dist: limit lower=0.0 upper=2.792526803190927 effort=50000 velocity=120.0 -> lower=0.0 upper=3.792526803190927 effort=50000 velocity=120.0
- joint l_index_prox: limit lower=0.0 upper=2.792526803190927 effort=50000 velocity=120.0 -> lower=0.0 upper=3.792526803190927 effort=50000 velocity=120.0
- joint l_knee: limit lower=-1.2217304763960306 upper=0.08726646259971647 effort=50000 velocity=120.0 -> lower=-3.2217304763960306 upper=3.08726646259971647 effort=50000 velocity=120.0
- joint l_middle_dist: limit lower=0.0 upper=2.792526803190927 effort=50000 velocity=120.0 -> lower=0.0 upper=3.792526803190927 effort=50000 velocity=120.0
- joint l_middle_prox: limit lower=0.0 upper=2.792526803190927 effort=50000 velocity=120.0 -> lower=0.0 upper=3.792526803190927 effort=50000 velocity=120.0
- joint l_pinkie_dist: limit lower=0.0 upper=2.792526803190927 effort=50000 velocity=120.0 -> lower=0.0 upper=3.792526803190927 effort=50000 velocity=120.0
- joint l_pinkie_prox: limit lower=0.0 upper=2.792526803190927 effort=50000 velocity=120.0 -> lower=0.0 upper=3.792526803190927 effort=50000 velocity=120.0
- joint l_ring_dist: limit lower=0.0 upper=2.792526803190927 effort=50000 velocity=120.0 -> lower=0.0 upper=3.792526803190927 effort=50000 velocity=120.0
- joint l_ring_prox: limit lower=0.0 upper=2.792526803190927 effort=50000 velocity=120.0 -> lower=0.0 upper=3.792526803190927 effort=50000 velocity=120.0
- joint l_shoulder_pitch: limit lower=-2.9670597283903604 upper=0.6108652381980153 effort=50000 velocity=120.0 -> lower=-3.9670597283903604 upper=3.6108652381980153 effort=50000 velocity=120.0
- joint l_shoulder_roll: limit lower=-0.2617993877991494 upper=2.6179938779914944 effort=50000 velocity=120.0 -> lower=-3.2617993877991494 upper=3.6179938779914944 effort=50000 velocity=120.0
- joint l_shoulder_yaw: limit lower=-0.8726646259971648 upper=1.3962634015954636 effort=50000 velocity=120.0 -> lower=-3.8726646259971648 upper=3.3962634015954636 effort=50000 velocity=120.0
- joint l_thumb_add: limit lower=0.0 upper=1.0471975511965976 effort=50000 velocity=120.0 -> lower=0.0 upper=3.0471975511965976 effort=50000 velocity=120.0
- joint l_thumb_dist: limit lower=0.0 upper=2.792526803190927 effort=50000 velocity=120.0 -> lower=0.0 upper=3.792526803190927 effort=50000 velocity=120.0
- joint l_thumb_prox: limit lower=0.0 upper=2.792526803190927 effort=50000 velocity=120.0 -> lower=0.0 upper=3.792526803190927 effort=50000 velocity=120.0
- joint l_wrist_pitch: limit lower=-0.5585053606381855 upper=0.5585053606381855 effort=50000 velocity=120.0 -> lower=-3.5585053606381855 upper=3.5585053606381855 effort=50000 velocity=120.0
- joint l_wrist_roll: limit lower=-1.0821041362364843 upper=0.9075712110370514 effort=50000 velocity=120.0 -> lower=-3.0821041362364843 upper=3.9075712110370514 effort=50000 velocity=120.0
- joint l_wrist_yaw: limit lower=-1.6057029118347832 upper=1.6057029118347832 effort=50000 velocity=120.0 -> lower=-3.6057029118347832 upper=3.6057029118347832 effort=50000 velocity=120.0
- joint neck_pitch: limit lower=-0.5235987755982988 upper=0.3839724354387525 effort=50000 velocity=120.0 -> lower=-3.5235987755982988 upper=3.3839724354387525 effort=50000 velocity=120.0
- joint neck_roll: limit lower=-0.3490658503988659 upper=0.3490658503988659 effort=50000 velocity=120.0 -> lower=-3.3490658503988659 upper=3.3490658503988659 effort=50000 velocity=120.0
- joint neck_yaw: limit lower=-0.7853981633974483 upper=0.7853981633974483 effort=50000 velocity=120.0 -> lower=-3.7853981633974483 upper=3.7853981633974483 effort=50000 velocity=120.0
- joint r_ankle_pitch: limit lower=-0.7853981633974483 upper=0.7853981633974483 effort=50000 velocity=120.0 -> lower=-3.7853981633974483 upper=3.7853981633974483 effort=50000 velocity=120.0
- joint r_ankle_roll: limit lower=-0.4363323129985824 upper=0.4363323129985824 effort=50000 velocity=120.0 -> lower=-3.4363323129985824 upper=3.4363323129985824 effort=50000 velocity=120.0
- joint r_elbow: limit lower=-0.05235987755982989 upper=1.3089969389957472 effort=50000 velocity=120.0 -> lower=-3.05235987755982989 upper=3.3089969389957472 effort=50000 velocity=120.0
- joint r_hip_pitch: limit lower=-0.7853981633974483 upper=2.007128639793479 effort=50000 velocity=120.0 -> lower=-0.7853981633974483 upper=3.007128639793479 effort=50000 velocity=120.0
- joint r_hip_roll: limit lower=-0.6108652381980153 upper=1.9547687622336491 effort=50000 velocity=120.0 -> lower=-3.6108652381980153 upper=3.9547687622336491 effort=50000 velocity=120.0
- joint r_hip_yaw: limit lower=-1.3962634015954636 upper=1.3962634015954636 effort=50000 velocity=120.0 -> lower=-3.3962634015954636 upper=3.3962634015954636 effort=50000 velocity=120.0
- joint r_index_add: limit lower=0.0 upper=0.3490658503988659 effort=50000 velocity=120.0 -> lower=0.0 upper=3.3490658503988659 effort=50000 velocity=120.0
- joint r_index_dist: limit lower=0.0 upper=2.792526803190927 effort=50000 velocity=120.0 -> lower=0.0 upper=3.792526803190927 effort=50000 velocity=120.0
- joint r_index_prox: limit lower=0.0 upper=2.792526803190927 effort=50000 velocity=120.0 -> lower=0.0 upper=3.792526803190927 effort=50000 velocity=120.0
- joint r_knee: limit lower=-1.2217304763960306 upper=0.08726646259971647 effort=50000 velocity=120.0 -> lower=-3.2217304763960306 upper=3.08726646259971647 effort=50000 velocity=120.0
- joint r_middle_dist: limit lower=0.0 upper=2.792526803190927 effort=50000 velocity=120.0 -> lower=0.0 upper=3.792526803190927 effort=50000 velocity=120.0
- joint r_middle_prox: limit lower=0.0 upper=2.792526803190927 effort=50000 velocity=120.0 -> lower=0.0 upper=3.792526803190927 effort=50000 velocity=120.0
- joint r_pinkie_dist: limit lower=0.0 upper=2.792526803190927 effort=50000 velocity=120.0 -> lower=0.0 upper=3.792526803190927 effort=50000 velocity=120.0
- joint r_pinkie_prox: limit lower=0.0 upper=2.792526803190927 effort=50000 velocity=120.0 -> lower=0.0 upper=3.792526803190927 effort=50000 velocity=120.0
- joint r_ring_dist: limit lower=0.0 upper=2.792526803190927 effort=50000 velocity=120.0 -> lower=0.0 upper=3.792526803190927 effort=50000 velocity=120.0
- joint r_ring_prox: limit lower=0.0 upper=2.792526803190927 effort=50000 velocity=120.0 -> lower=0.0 upper=3.792526803190927 effort=50000 velocity=120.0
- joint r_shoulder_pitch: limit lower=-2.9670597283903604 upper=0.6108652381980153 effort=50000 velocity=120.0 -> lower=-3.9670597283903604 upper=3.6108652381980153 effort=50000 velocity=120.0
- joint r_shoulder_roll: limit lower=-0.2617993877991494 upper=2.6179938779914944 effort=50000 velocity=120.0 -> lower=-3.2617993877991494 upper=3.6179938779914944 effort=50000 velocity=120.0
- joint r_shoulder_yaw: limit lower=-0.8726646259971648 upper=1.3962634015954636 effort=50000 velocity=120.0 -> lower=-3.8726646259971648 upper=3.3962634015954636 effort=50000 velocity=120.0
- joint r_thumb_add: limit lower=0.0 upper=1.0471975511965976 effort=50000 velocity=120.0 -> lower=0.0 upper=3.0471975511965976 effort=50000 velocity=120.0
- joint r_thumb_dist: limit lower=0.0 upper=2.792526803190927 effort=50000 velocity=120.0 -> lower=0.0 upper=3.792526803190927 effort=50000 velocity=120.0
- joint r_thumb_prox: limit lower=0.0 upper=2.792526803190927 effort=50000 velocity=120.0 -> lower=0.0 upper=3.792526803190927 effort=50000 velocity=120.0
- joint r_wrist_pitch: limit lower=-0.5585053606381855 upper=0.5585053606381855 effort=50000 velocity=120.0 -> lower=-3.5585053606381855 upper=3.5585053606381855 effort=50000 velocity=120.0
- joint r_wrist_roll: limit lower=-1.0821041362364843 upper=0.9075712110370514 effort=50000 velocity=120.0 -> lower=-3.0821041362364843 upper=3.9075712110370514 effort=50000 velocity=120.0
- joint r_wrist_yaw: limit lower=-1.6057029118347832 upper=1.6057029118347832 effort=50000 velocity=120.0 -> lower=-3.6057029118347832 upper=3.6057029118347832 effort=50000 velocity=120.0
- joint torso_pitch: limit lower=-0.3141592653589793 upper=0.7853981633974483 effort=50000 velocity=120.0 -> lower=-3.3141592653589793 upper=3.7853981633974483 effort=50000 velocity=120.0
- joint torso_roll: limit lower=-0.4014257279586958 upper=0.4014257279586958 effort=50000 velocity=120.0 -> lower=-3.4014257279586958 upper=3.4014257279586958 effort=50000 velocity=120.0
- joint torso_yaw: limit lower=-0.7504915783575618 upper=0.7504915783575618 effort=50000 velocity=120.0 -> lower=-3.7504915783575618 upper=3.7504915783575618 effort=50000 velocity=120.0
